Commit message: Simulate all last

File: src/sim_pkg/urdf/gimbal_camera_attachment.urdf (robot description, URDF)
Before this commit: robot gimbal_camera_attachment, 5 links, 4 joints
Joints:
- joint gimbal_pitch_joint: limit lower=-0.6109 upper=1.5708 effort=2 velocity=2 -> lower=-1.5708 upper=0.6109 effort=2 velocity=2
