Commit message: 修正URDF参数，更新RVIZ

File: src/sim_pkg/urdf/smartcar.urdf (robot description, URDF)
Before this commit: robot smartcar, 13 links, 12 joints
Links:
- link base_link: geometry collision box size=0.32 .15 .05; visual box size=0.32 .15 .05
- link landing_pad: geometry collision box size=0.25 0.30 0.012; visual box size=0.25 0.30 0.012
- link left_back_wheel: geometry collision cylinder length=.04 radius=0.05; visual cylinder length=.04 radius=0.05
- link left_front_wheel: geometry collision cylinder length=.04 radius=0.05; visual cylinder length=.04 radius=0.05
- link right_back_wheel: geometry collision cylinder length=.02 radius=0.025; visual cylinder length=.04 radius=0.05
- link right_front_wheel: geometry collision cylinder length=.04 radius=0.05; visual cylinder length=.04 radius=0.05
Joints:
- joint left_back_wheel_joint: origin xyz=-0.08 -0.1 -0.03 rpy=0 1.57075 0.785398 -> xyz=-0.095 -0.11 -0.03 rpy=0 1.57075 0
- joint left_front_wheel_joint: origin xyz=-0.08 0.1 -0.03 rpy=0 1.57075 -0.785398 -> xyz=-0.095 0.11 -0.03 rpy=0 1.57075 0
- joint right_back_wheel_joint: origin xyz=0.08 -0.1 -0.03 rpy=0 1.57075 -0.785398 -> xyz=0.095 -0.11 -0.03 rpy=0 1.57075 0
- joint right_front_wheel_joint: origin xyz=0.08 0.1 -0.03 rpy=0 1.57075 0.785398 -> xyz=0.095 0.11 -0.03 rpy=0 1.57075 0

Commit message: 优化小车URDF，更新小车与gazebo 联动launch文件，更新rviz配置文件

File: src/sim_pkg/urdf/smartcar.urdf (robot description, URDF)
Before this commit: robot smartcar, 13 links, 12 joints
Links:
- link right_back_wheel: geometry collision cylinder length=.04 radius=0.05; visual cylinder length=.04 radius=0.05
Joints:
- joint base_footprint_joint: origin xyz=0 0 0.082 rpy=0 0 0 -> xyz=0 0 0.082 rpy=0 0 -1.57075

Commit message: 重构小车仿真控制器，支持全向移动

File: src/sim_pkg/urdf/smartcar.urdf (robot description, URDF)
Before this commit: robot smartcar, 13 links, 12 joints
Links:
- link landing_pad: mass 0.1 -> 1.0
- link left_back_wheel: mass 0.1 -> 0.5
- link left_front_wheel: mass 0.1 -> 0.5
- link right_back_wheel: mass 0.1 -> 0.5
- link right_front_wheel: mass 0.1 -> 0.5

Commit message: 更新launch文件相关仿真参数

File: src/sim_pkg/urdf/smartcar.urdf (robot description, URDF)
Before this commit: robot smartcar, 13 links, 12 joints
Links:
- link base_link: mass 1.5 -> 2.5
- link landing_pad: mass 1.0 -> 1.5; geometry collision box size=0.35 0.35 0.012; visual box size=0.35 0.35 0.012
- link left_back_wheel: mass 0.5 -> 0.8
- link left_front_wheel: mass 0.5 -> 0.8
- link right_back_wheel: mass 0.5 -> 0.8
- link right_front_wheel: mass 0.5 -> 0.8
Joints:
- joint left_back_wheel_joint: limit effort=100 velocity=100 -> effort=50 velocity=50; type continuous -> fixed
- joint left_front_wheel_joint: limit effort=100 velocity=100 -> effort=50 velocity=50; type continuous -> fixed
- joint right_back_wheel_joint: limit effort=100 velocity=100 -> effort=50 velocity=50; type continuous -> fixed
- joint right_front_wheel_joint: limit effort=100 velocity=100 -> effort=50 velocity=50; type continuous -> fixed

Commit message: 优化仿真参数

File: src/sim_pkg/urdf/smartcar.urdf (robot description, URDF)
Before this commit: robot smartcar, 13 links, 12 joints
Links:
- removed link landing_pad_stick_1
- removed link landing_pad_stick_2
- removed link landing_pad_stick_3
- removed link landing_pad_stick_4
- link base_link: geometry collision box size=0.32 0.15 .15; visual box size=0.32 .15 .05
- link head: geometry visual box size=.02 .03 .03
- link left_back_wheel: geometry visual cylinder length=.04 radius=0.05
- link left_front_wheel: geometry visual cylinder length=.04 radius=0.05
- link right_back_wheel: geometry visual cylinder length=.04 radius=0.05
- link right_front_wheel: geometry visual cylinder length=.04 radius=0.05
Joints:
- removed joint landing_pad_stick_1_joint
- removed joint landing_pad_stick_2_joint
- removed joint landing_pad_stick_3_joint
- removed joint landing_pad_stick_4_joint

Commit message: 优化仿真模型参数，加入Gazebo-attach-link插件，加入仿真环境中的机器人位置复位脚本

File: src/sim_pkg/urdf/smartcar.urdf (robot description, URDF)
Before this commit: robot smartcar, 9 links, 8 joints
Links:
- link base_link: mass 2.5 -> 1.2; geometry collision box size=0.45 0.30 .15; visual box size=0.32 .15 .05
- link landing_pad: mass 1.5 -> 12.5

Commit message: 仿真环境以及部分参数调整

File: src/sim_pkg/urdf/smartcar.urdf (robot description, URDF)
Before this commit: robot smartcar, 9 links, 8 joints
Joints:
- joint landing_pad_joint: origin xyz=0 0 0.06 -> xyz=0 0 0.06 rpy=0 0 1.57
